File: H_Bridge/H_Bridge.kicad_sch (KiCad schematic)
At the start: 28 parts, among them IC1 FAN7382N, IC2 FAN7382N, J1 TB_1X2, Q1 IRFZ44N, Q2 IRFZ44N, Q3 IRFZ44N, Q4 IRFZ44N, U3 CD4093B

Commit message: new
Parts:
- removed JP2: Jumper, symbol EESTN5:Jumper
- removed U3: CD4093B, symbol Logic_Gate:CD4093B
- added C6, C7, C8: C, symbol EESTN5:C
- added J2: CONN_01X02, symbol MacroLib:CONN_01X02
- added R12, R13, R14: R, symbol EESTN5:R
- added U1, U2: CD4093B, symbol Logic_Gate:CD4093B
Connections:
- net GND: now also C6.2, C7.2, C8.2
- net at R2.1: now also U1.1 (A)
- net at C2.1, R2.2: now also U1.2 (B)
- net VDD: now reaches C3.1, IC1.1 (VCC), R1.1
- net VDD: now also C4.1, IC2.1 (VCC), R7.1; no longer JP1.1 (A)
- new net: C8.1, R14.2, U2.9 (F)
- new net: R12.1, U1.8 (E)
- new net: C6.1, R12.2, U1.9 (F)
- new net: J2.2 (P2), U1.14 (VDD), U2.14 (VDD)
- new net: J2.1 (P1), U1.7 (VSS), U2.7 (VSS)
- new net: U1.10 (L), U1.12 (G), U1.13 (H)
- new net: C7.1, R13.2, U2.2 (B)
- new net: U1.3 (J), U1.5 (C), U1.6 (D)
- new net: R13.1, U2.1 (A)
- new net: U2.3 (J), U2.5 (C), U2.6 (D)
- new net: R14.1, U2.8 (E)
- new net: U2.10 (L), U2.12 (G), U2.13 (H)
Other:
- moved on the sheet: C3, C4, JP1
